Commit message: update

File: src/earth_description/urdf/earthfibo.xacro (robot description, xacro)
@@ -1,5 +1,12 @@
 <?xml version="1.0"?>
 <robot name="earthfibo" xmlns:xacro="http://www.ros.org/wiki/xacro">
+<!--การสร้างหุ่นหลักๆ จะมี3 ส่วนประกอบหลักคือ 1.visual ถ้าเปรียบเทียบง่ายๆ visual คือ วิญญาณ 2.collision คือ กายหยาบ 3.inertial คือการขยับทำสิ่งต่างๆ
+การจะต้องมี3ส่วนประกอบ กรณีขาดไปอย่างใดอย่างหนึ่ง จะทำให้หุ่นเรา้เจอปัญหาได้ เช่น กรณีหุ่นชนสิ่งกีดขวาง ถ้าไม่มี collision มันจะทะลุผ่านไปเลย
+การเขียน visual collision สามารถสร้างรูปทรงต่างๆได้ เช่น ทรงกลม สี่เหลี่ยม
+สิ่งที่ขาดไม่ได้เลยในการทำหุ่นยนต์คือ joint  joint จะเป็นตัวเชื่อมส่วนประกอบต่างๆให้หุ่นสามารถเคลื่อนที่ได้
+สิ่งสำคัญในการออกแบบหุ่นคือ
+ -->
 <link name="body">
+<!--สร้างโครงหุ่น-->
     <visual>
           <geometry>
@@ -23,4 +30,5 @@
    </collision>
     </link>
+     <!--สร้างล้อซ้าย-->
      <link name="left_wheel">
        <visual>
@@ -53,4 +61,5 @@
         <dynamics damping='0.3'/>
      </joint>
+    <!--สร้างล้อขวา-->
     <link name="right_wheel">
        <visual>
@@ -83,34 +92,5 @@
         <dynamics damping='0.3'/>
      </joint>
-<!-->
-   <link name="fwheel_attach">
-       <visual>
-         <geometry>
-           <cylinder length="0.060" radius="0.023"/>
-         </geometry>
-         <origin rpy="0 0 0" xyz="0.13 0 0.08"/>
-         <material name="white">
-           <color rgba="1 1 1 1"/>
-         </material>
-       </visual>
-        <collision name="collision">
-          <origin rpy="0 0 0" xyz="0.13 0 0.08"/>
-          <geometry>
-              <cylinder length="0.060" radius="0.023"/>
-          </geometry>
-        </collision>
-        <inertial>
-     <origin xyz="0 0 0" rpy="0 0 0"/>
-     <mass value="1"/>
-     <inertia ixx="0.1"  ixy="0"  ixz="0" iyy="0.1" iyz="0" izz="0.1" />
-   </inertial>
-     </link>
-     <joint name="base_to_fattach" type="continuous">
-       <parent link="body"/>
-       <child link="fwheel_attach"/>
-       <origin xyz="0 0 0" rpy="0 0 0"/>
-         <axis xyz="0 1 0"/>
-     </joint>
- <-->
+     <!--สร้างล้อหน้า-->
      <link name="fwheel">
        <visual>
@@ -141,4 +121,5 @@
         <axis xyz="0 1 0"/>
      </joint>
+   <!--สร้างกล้อง-->
   <joint name="camera_joint" type="fixed">
     <origin xyz="0.105 0 0.1" rpy="0 0 0" />
@@ -216,4 +197,5 @@
     <child link="hokuyo_link"/>
   </joint>
+  <!--สร้างlidar sensor-->
   <!-- Hokuyo Laser -->
   <link name="hokuyo_link">
@@ -272,4 +254,5 @@
     </sensor>
   </gazebo>
+<!--plugin controller-->
 <gazebo>
   <plugin name="differential_drive_controller" filename="libgazebo_ros_diff_drive.so">
